File: hardware/Praticenew.kicad_pcb (KiCad board)
At the start: 4 copper layers, 82 x 49 mm, 14 parts, among them U1 MAX30102, U2 Untitled

Commit message: Switch to 2-layer stackup, 10k pull-ups, fix OLED value
Co-Authored-By: Claude Opus 5.5 <noreply@anthropic.com>
Claude-Session: https://claude.ai/code/session_01LM6eX8d7eE2LMZS3NBMFqz
Parts:
- R1, R2, R3: value 1k -> 10k
- U2: value Untitled -> OLED
Other:
- copper layers 4 -> 2
Changed lines of the file:
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@@
 	(layers
 		(0 "F.Cu" signal "Front")
-		(4 "In1.Cu" signal)
-		(6 "In2.Cu" signal)
 		(2 "B.Cu" signal "Back")
 		(13 "F.Paste" user)
@@
 			(layer "dielectric 1"
 				(type "core")
-				(thickness 0.480066)
-				(material "FR4")
-				(epsilon_r 4.5)
-				(loss_tangent 0.02)
-			)
-			(layer "In1.Cu"
-				(type "copper")
-				(thickness 0.035)
-			)
-			(layer "dielectric 2"
-				(type "prepreg")
-				(thickness 0.480066)
-				(material "FR4")
-				(epsilon_r 4.5)
-				(loss_tangent 0.02)
-			)
-			(layer "In2.Cu"
-				(type "copper")
-				(thickness 0.035)
-			)
-			(layer "dielectric 3"
-				(type "core")
-				(thickness 0.480066)
+				(thickness 1.510198)
 				(material "FR4")
 				(epsilon_r 4.5)
@@
 			)
 		)
-		(property "Value" "Untitled"
+		(property "Value" "OLED"
 			(at 0 1 0)
 			(unlocked yes)
@@
 			)
 		)
-		(property "Value" "1k"
+		(property "Value" "10k"
 			(at 3.81 2.37 90)
 			(layer "F.Fab")
@@
 			)
 		)
-		(property "Value" "1k"
+		(property "Value" "10k"
 			(at 3.81 2.37 90)
 			(layer "F.Fab")
@@
 			)
 		)
-		(property "Value" "1k"
+		(property "Value" "10k"
 			(at 3.81 2.37 90)
 			(layer "F.Fab")
