File: hardware/Praticenew.kicad_sch (KiCad schematic)
At the start: 14 parts, among them SW1 SW_Push, SW2 SW_Push, SW3 SW_Push, U1 MAX30102, U2 SSD1306

Commit message: Sync schematic to 10k pull-ups, add DRC result
Co-Authored-By: Claude Opus 5.5 <noreply@anthropic.com>
Claude-Session: https://claude.ai/code/session_01LM6eX8d7eE2LMZS3NBMFqz
Parts:
- R1, R2, R3: value 1k -> 10k
Other:
- moved on the sheet: A1, C1, C2, C3, D1, R1, R2, R3, R4, SW1, SW2, SW3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
